File: F3_UI_Board/F3_UI_Board.kicad_pcb (KiCad board)
At the start: 2 copper layers, 72 x 47.5 mm, 37 parts, among them J1 Conn_ARM_JTAG_SWD_10, J2 Conn_02x05_Odd_Even, SW1 SW_Push, SW2 SW_Push, SW3 SW_Push, U1 STM32F303K8Tx, Y1 8M RH100-8.000-20-3050-EXT-TR

Commit message: [fix] pull up
Parts:
- added R11: 10k, Resistor_SMD:R_0603_1608Metric, F.Cu at (87.8, 132.6)
- added R12: 10k, Resistor_SMD:R_0603_1608Metric, F.Cu at (91.9, 132.6)
- moved C9 0.06 mm to (89.8, 135.8), turned to 90 degrees
Connections:
- C9 pad 1: /ADC1_IN4 -> Net-(C9-Pad1)
- C9 pad 2: Net-(C9-Pad2) -> /ADC1_IN4
- TP3 pad 1: Net-(C9-Pad2) -> Net-(C9-Pad1)
Routing:
- net Net-(C9-Pad2): track 5.03 -> 0.00 mm
- net Net-(C9-Pad1): track 0.00 -> 5.03 mm
- net /ADC1_IN4: track 43.0 -> 45.6 mm
- net /VDD_MCU: track 231.5 -> 233.3 mm
- net GND: track 397.0 -> 398.7 mm
