File: F3_UI_Board/F3_UI_Board.sch (KiCad schematic (older format))
At the start: 37 parts, among them J1 Conn_ARM_JTAG_SWD_10, J2 Conn_02x05_Odd_Even, SW1 SW_Push, SW2 SW_Push, SW3 SW_Push, U1 STM32F303K8Tx, Y1 8M RH100-8.000-20-3050-EXT-TR

Commit message: [fix] pull up
Parts:
- added R11, R12: 10k, Resistor_SMD:R_0603_1608Metric, symbol Device:R
Connections:
- net ADC1_IN4: now also C9.2, R11.1, R12.2; no longer C9.1
- net GND: now also R12.1
- net VDD_MCU: now also R11.2
- net at TP3.1: now also C9.1; no longer C9.2
Other:
- moved on the sheet: C9, TP3
Changed lines of the file:
@@
 L Device:C_Small C9
 U 1 1 5E8249AA
-P 10300 5400
-F 0 "C9" H 10200 5300 50  0000 C CNN
-F 1 "0.1u" H 10200 5500 50  0000 C CNN
-F 2 "Capacitor_SMD:C_0603_1608Metric" H 10300 5400 50  0001 C CNN
-F 3 "~" H 10300 5400 50  0001 C CNN
-	1    10300 5400
-	-1   0    0    1
-$EndComp
-Text Label 10300 5600 3    50   ~ 0
+P 10550 5350
+F 0 "C9" H 10450 5250 50  0000 C CNN
+F 1 "0.1u" H 10450 5450 50  0000 C CNN
+F 2 "Capacitor_SMD:C_0603_1608Metric" H 10550 5350 50  0001 C CNN
+F 3 "~" H 10550 5350 50  0001 C CNN
+	1    10550 5350
+	0    1    1    0
+$EndComp
+Text Label 10100 5350 1    50   ~ 0
 ADC1_IN4
-Wire Wire Line
-	10300 5600 10300 5500
-Wire Wire Line
-	10300 5300 10300 5100
 $Comp
 L Connector:TestPoint TP3
 U 1 1 5E82D2D1
-P 10300 5100
-F 0 "TP3" H 10358 5218 50  0000 L CNN
-F 1 "TestPoint" H 10358 5127 50  0000 L CNN
-F 2 "Connector_Pin:Pin_D1.0mm_L10.0mm" H 10500 5100 50  0001 C CNN
-F 3 "~" H 10500 5100 50  0001 C CNN
-	1    10300 5100
+P 10650 4900
+F 0 "TP3" H 10708 5018 50  0000 L CNN
+F 1 "TestPoint" H 10708 4927 50  0000 L CNN
+F 2 "Connector_Pin:Pin_D1.0mm_L10.0mm" H 10850 4900 50  0001 C CNN
+F 3 "~" H 10850 4900 50  0001 C CNN
+	1    10650 4900
 	1    0    0    -1
 $EndComp
@@
 Wire Wire Line
 	1000 4500 1000 4350
+$Comp
+L Device:R R11
+U 1 1 5E727C61
+P 10300 5000
+F 0 "R11" H 10230 4954 50  0000 R CNN
+F 1 "10k" H 10230 5045 50  0000 R CNN
+F 2 "Resistor_SMD:R_0603_1608Metric" V 10230 5000 50  0001 C CNN
+F 3 "~" H 10300 5000 50  0001 C CNN
+	1    10300 5000
+	-1   0    0    1
+$EndComp
+$Comp
+L Device:R R12
+U 1 1 5E73D310
+P 10300 5700
+F 0 "R12" H 10230 5654 50  0000 R CNN
+F 1 "10k" H 10230 5745 50  0000 R CNN
+F 2 "Resistor_SMD:R_0603_1608Metric" V 10230 5700 50  0001 C CNN
+F 3 "~" H 10300 5700 50  0001 C CNN
+	1    10300 5700
+	-1   0    0    1
+$EndComp
+Wire Wire Line
+	10300 5550 10300 5350
+Wire Wire Line
+	10650 4900 10650 5350
+Wire Wire Line
+	10450 5350 10300 5350
+Connection ~ 10300 5350
+Wire Wire Line
+	10300 5350 10300 5150
+Wire Wire Line
+	10300 5350 10100 5350
+$Comp
+L power:GND #PWR019
+U 1 1 5E75CA01
+P 10300 5950
+F 0 "#PWR019" H 10300 5700 50  0001 C CNN
+F 1 "GND" H 10305 5777 50  0000 C CNN
+F 2 "" H 10300 5950 50  0001 C CNN
+F 3 "" H 10300 5950 50  0001 C CNN
+	1    10300 5950
+	1    0    0    -1
+$EndComp
+Wire Wire Line
+	10300 5950 10300 5850
+Text Label 10300 4750 1    50   ~ 0
+VDD_MCU
+Wire Wire Line
+	10300 4750 10300 4850
 $EndSCHEMATC
